File: hardware/main_pcb_hw5/vselect.kicad_sch (KiCad schematic)
At the start: 5 parts, among them U1 TPS2113PW

Commit message: Changed 0402 components to 0603
 - Also tweaked name in board graphics to make it clear this isn't a
   vanilla board.
Parts:
- C2, C3, C4: footprint Capacitor_SMD:C_0402_1005Metric_Pad0.74x0.62mm_HandSolder -> Capacitor_SMD:C_0603_1608Metric_Pad1.08x0.95mm_HandSolder
- R2: footprint Resistor_SMD:R_0402_1005Metric_Pad0.72x0.64mm_HandSolder -> Resistor_SMD:R_0603_1608Metric_Pad0.98x0.95mm_HandSolder
